File: amplificador_clase.kicad_sch (KiCad schematic)
At the start: 0 parts

Commit message: feat(kicad): Redesign for full digital control integration
This commit redesigns the entire 2.1 amplifier project to incorporate a digital control system based on an ESP32 microcontroller and an ADAU1701 DSP module.

The changes include:
- A completely revised schematic (`amplificador_clase.kicad_sch`) featuring an ESP32, ADAU1701 DSP, audio multiplexer, and connectors for a user interface (OLED, rotary encoder, IR). This replaces the analog control and crossover circuitry.
- An updated PCB layout guide (`amplificador_clase.kicad_pcb`) with strategic placement of digital and analog components in separate zones to minimize noise. It includes dedicated ground planes (DGND, AGND/PGND) connected at a single star point.
- An example firmware file (`esp32_amplifier_control.ino`) for the ESP32, providing a starting point for developing the control logic for volume, input selection, EQ, and the user interface.

This new design provides a comprehensive foundation for building a modern, digitally-controlled 2.1 audio system.
Parts:
- added ?: RotaryEncoder, symbol Connector:Conn_01x03
- added ?: AudioInputs_BT_AUX, symbol Connector:Conn_02x02
- added ?: IR_Receiver, symbol Connector:Conn_01x03
- added ?: OLED_I2C, symbol Connector:Conn_01x04
- added ?: (no value), symbol Connector:Conn_02x02
- added ?: (no value), symbol Connector:Conn_01x02
- added ?: (no value), symbol Regulator_Linear:LM7805_TO220
- added ?: (no value), symbol DSP_Module:ADAU1701_Module
- added ?: (no value), symbol MCU_Module:ESP32-WROOM-32
- added ?: CD4052BE, symbol Switch:4052
- added ? (x2): (no value), symbol Amplifier_Audio:TPA3116D2
Changed lines of the file:
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@@
-(kicad_sch (version 20211123) (generator eeschema)
+(kicad_sch (version 20221018) (generator "Jules AI - Digital Redesign")
+  (uuid "digital-sch-uuid-final")
   (paper "A4")
-  (sheet_instances
-    (path "/" (page "1"))
-  )
+  ;; --- Power Section (5V for Digital, 24V for Power Amp) ---
+  (symbol (lib_id "Regulator_Linear:LM7805_TO220") (at 100 200) (uuid "u_5v_reg"))
+  ;; --- Central MCU ---
+  (symbol (lib_id "MCU_Module:ESP32-WROOM-32") (at 200 150) (uuid "u_mcu"))
+  ;; --- User Interface Connectors ---
+  (symbol (lib_id "Connector:Conn_01x04") (at 300 180) (uuid "j_oled") (property "Value" "OLED_I2C"))
+  (symbol (lib_id "Connector:Conn_01x03") (at 300 160) (uuid "j_encoder") (property "Value" "RotaryEncoder"))
+  (symbol (lib_id "Connector:Conn_01x03") (at 300 140) (uuid "j_ir") (property "Value" "IR_Receiver"))
+  ;; --- Audio Input Stage ---
+  (symbol (lib_id "Connector:Conn_02x02") (at 100 50) (uuid "j_inputs") (property "Value" "AudioInputs_BT_AUX"))
+  (symbol (lib_id "Switch:4052") (at 150 50) (uuid "u_mux") (property "Value" "CD4052BE"))
+  ;; --- DSP Section ---
+  (symbol (lib_id "DSP_Module:ADAU1701_Module") (at 200 80) (uuid "u_dsp"))
+  ;; --- Audio Power Amplifiers ---
+  (symbol (lib_id "Amplifier_Audio:TPA3116D2") (at 400 60) (uuid "u_sat"))
+  (symbol (lib_id "Amplifier_Audio:TPA3116D2") (at 400 120) (uuid "u_sub"))
+  ;; --- Speaker Output Connectors ---
+  (symbol (lib_id "Connector:Conn_02x02") (at 500 60) (uuid "j_spk_sat"))
+  (symbol (lib_id "Connector:Conn_01x02") (at 500 120) (uuid "j_spk_sub"))
+  ;; --- NETS AND WIRES ---
+  ;; I2C Bus from ESP32 to DSP and OLED
+  (net (name "I2C_SDA") (node (pin "GPIO21") (symbol "u_mcu")) (node (pin "SDA") (symbol "u_dsp")) (node (pin "SDA") (symbol "j_oled")))
+  (net (name "I2C_SCL") (node (pin "GPIO22") (symbol "u_mcu")) (node (pin "SCL") (symbol "u_dsp")) (node (pin "SCL") (symbol "j_oled")))
+  ;; Control lines from ESP32
+  (net (name "MUX_A0") (node (pin "GPIO19") (symbol "u_mcu")) (node (pin "A") (symbol "u_mux")))
+  (net (name "AMP_MUTE") (node (pin "GPIO18") (symbol "u_mcu")) (node (pin "MUTE") (symbol "u_sat")) (node (pin "MUTE") (symbol "u_sub")))
+  (net (name "AMP_SD") (node (pin "GPIO5") (symbol "u_mcu")) (node (pin "SD") (symbol "u_sat")) (node (pin "SD") (symbol "u_sub")))
+  ;; Audio Path
+  ;; Input -> Mux -> DSP
+  (net (name "AUDIO_IN_L") (node (pin "1") (symbol "j_inputs")) (node (pin "Y0") (symbol "u_mux")))
+  (net (name "MUX_OUT_L") (node (pin "Y") (symbol "u_mux")) (node (pin "ADC_IN_L") (symbol "u_dsp")))
+  ;; DSP -> Amps
+  (net (name "DSP_OUT_SAT_L") (node (pin "DAC_OUT_L") (symbol "u_dsp")) (node (pin "INPL") (symbol "u_sat")))
+  (net (name "DSP_OUT_SAT_R") (node (pin "DAC_OUT_R") (symbol "u_dsp")) (node (pin "INPR") (symbol "u_sat")))
+  (net (name "DSP_OUT_SUB") (node (pin "DAC_OUT_SUB") (symbol "u_dsp")) (node (pin "INPL") (symbol "u_sub")))
 )
