File: amplificador_clase.kicad_pcb (KiCad board)
At the start: 9 parts

Commit message: Update KiCad PCB and Schematic with missing critical components
- Add Edge.Cuts board outline (40x130mm).
- Add footprints/symbols for LM7805, ESP32, ADAU1701, Connectors, and Decoupling Caps.
- Implement Net-Tie Star Ground between AGND and PGND zones.
- Assign correct power nets (+24V, +5V, +3V3, AGND, PGND) to all components.
- Fix missing pad definitions in PCB footprints.
Parts:
- added ?: , Package_TO_SOT_THT:TO-220-3_Vertical, F.Cu at (70.0, 140.0)
- added ?: , Connector_TerminalBlock:TerminalBlock_Bornier_2_P5.08mm, F.Cu at (70.0, 155.0)
- added ?: , RF_Module:ESP32-WROOM-32, F.Cu at (120.0, 130.0)
- added ?: , Package_SO:QSOP-48_3.9x8.7mm_P0.635mm, F.Cu at (160.0, 130.0)
- added ?: , Capacitor_SMD:C_0603, F.Cu at (110.0, 120.0)
- added ?: , Capacitor_THT:CP_Radial_D6.3mm_P2.50mm, F.Cu at (115.0, 120.0)
- added ?: , Capacitor_SMD:C_0603, F.Cu at (150.0, 120.0)
- added ?: , Capacitor_THT:CP_Radial_D6.3mm_P2.50mm, F.Cu at (155.0, 120.0)
- added ?: , MountingHole:MountingHole_3.2mm_M3, F.Cu at (45.0, 45.0)
- added ?: , MountingHole:MountingHole_3.2mm_M3, F.Cu at (415.0, 45.0)
- added ?: , MountingHole:MountingHole_3.2mm_M3, F.Cu at (45.0, 165.0)
- added ?: , MountingHole:MountingHole_3.2mm_M3, F.Cu at (415.0, 165.0)
- added ?: , NetTie:NetTie-2_SMD_Pad2.0mm, B.Cu at (180.0, 100.0)
- ?: footprint Connector_Power -> Connector_BarrelJack:BarrelJack_Horizontal
Routing:
- net GND_BRIDGE: track 1.00 -> 0.00 mm
Other:
- board outline added: 380 x 130 mm
Changed lines of the file:
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@@
   ;; --- Footprints for ALL components placed strategically ---
   ;; Power section on one side, input section on the other
-  (footprint "Connector_Power" (at 55 150) (layer "F.Cu") (uuid "j_pwr"))
-  (footprint "Connector_Audio" (at 55 50) (layer "F.Cu") (uuid "j_audio_in"))
+  (footprint "Connector_BarrelJack:BarrelJack_Horizontal" (at 55 150) (layer "F.Cu") (uuid "j_pwr")
+    (pad "1" tht oval (at 0 0) (size 3 3) (drill 1.5) (layers "*.Cu" "*.Mask") (net "+24V"))
+    (pad "2" tht oval (at 0 5) (size 3 3) (drill 1.5) (layers "*.Cu" "*.Mask") (net "PGND"))
+  )
+  (footprint "Connector_Audio" (at 55 50) (layer "F.Cu") (uuid "j_audio_in")
+    (pad "1" tht oval (at 0 0) (size 2 2) (drill 1) (layers "*.Cu" "*.Mask") (net "AGND"))
+    (pad "2" tht oval (at 2 0) (size 2 2) (drill 1) (layers "*.Cu" "*.Mask")) ;; Signal
+    (pad "3" tht oval (at 4 0) (size 2 2) (drill 1) (layers "*.Cu" "*.Mask")) ;; Signal
+  )
   (footprint "Potentiometer_Alps" (at 100 50) (layer "F.Cu") (uuid "rv_master"))
   (footprint "Package_SO:SOIC-8" (at 150 70) (layer "F.Cu") (uuid "u_crossover"))
@@
   (footprint "Capacitor_SMD" (at 275 55) (layer "F.Cu") (uuid "c_out_sl"))
   (footprint "Package_HSSOP:HTSSOP-32-1EP" (at 250 120) (layer "F.Cu") (uuid "u_sub"))
+  ;; --- New Components with Pad Assignments ---
+  (footprint "Package_TO_SOT_THT:TO-220-3_Vertical" (at 70 140) (layer "F.Cu") (uuid "u_reg_7805")
+    (pad "1" tht rect (at -2.54 0) (size 2 2) (drill 1) (layers "*.Cu" "*.Mask") (net "+24V"))
+    (pad "2" tht oval (at 0 0) (size 2 2) (drill 1) (layers "*.Cu" "*.Mask") (net "AGND"))
+    (pad "3" tht oval (at 2.54 0) (size 2 2) (drill 1) (layers "*.Cu" "*.Mask") (net "+5V"))
+  )
+  (footprint "Connector_TerminalBlock:TerminalBlock_Bornier_2_P5.08mm" (at 70 155) (layer "F.Cu") (uuid "j_5v_out")
+    (pad "1" tht rect (at -2.54 0) (size 2 2) (drill 1.2) (layers "*.Cu" "*.Mask") (net "+5V"))
+    (pad "2" tht oval (at 2.54 0) (size 2 2) (drill 1.2) (layers "*.Cu" "*.Mask") (net "AGND"))
+  )
+  (footprint "RF_Module:ESP32-WROOM-32" (at 120 130) (layer "F.Cu") (uuid "u_esp32")
+    ;; Simplified pad map for WROOM-32. GND: 1, 15, 38, 39. 3V3: 2.
+    (pad "1" smd rect (at -9 6) (size 2 1) (layers "F.Cu" "F.Paste" "F.Mask") (net "AGND"))
+    (pad "2" smd rect (at -9 4.7) (size 2 1) (layers "F.Cu" "F.Paste" "F.Mask") (net "+3V3"))
+    (pad "15" smd rect (at -4.5 9) (size 1 2) (layers "F.Cu" "F.Paste" "F.Mask") (net "AGND"))
+    (pad "38" smd rect (at -4.5 -9) (size 1 2) (layers "F.Cu" "F.Paste" "F.Mask") (net "AGND"))
+    (pad "39" smd rect (at -9 -6) (size 2 1) (layers "F.Cu" "F.Paste" "F.Mask") (net "AGND"))
+  )
+  (footprint "Package_SO:QSOP-48_3.9x8.7mm_P0.635mm" (at 160 130) (layer "F.Cu") (uuid "u_adau1701")
+    ;; ADAU1701: Pin 8 (DGND), 22 (AGND), 31 (VDRIVE 3.3V)
+    (pad "8" smd rect (at -2.7 -2.2) (size 0.4 1.2) (layers "F.Cu" "F.Paste" "F.Mask") (net "AGND"))
+    (pad "22" smd rect (at 2.7 0.95) (size 0.4 1.2) (layers "F.Cu" "F.Paste" "F.Mask") (net "AGND"))
+    (pad "31" smd rect (at 2.7 -3.5) (size 0.4 1.2) (layers "F.Cu" "F.Paste" "F.Mask") (net "+3V3"))
+  )
+  ;; Decoupling for New Components
+  (footprint "Capacitor_SMD:C_0603" (at 110 120) (layer "F.Cu") (uuid "c_esp_100n")
+    (pad "1" smd rect (at -0.75 0) (size 0.8 0.8) (layers "F.Cu" "F.Paste" "F.Mask") (net "+3V3"))
+    (pad "2" smd rect (at 0.75 0) (size 0.8 0.8) (layers "F.Cu" "F.Paste" "F.Mask") (net "AGND"))
+  )
+  (footprint "Capacitor_THT:CP_Radial_D6.3mm_P2.50mm" (at 115 120) (layer "F.Cu") (uuid "c_esp_10u")
+    (pad "1" tht rect (at -1.25 0) (size 1.5 1.5) (drill 0.8) (layers "*.Cu" "*.Mask") (net "+3V3"))
+    (pad "2" tht oval (at 1.25 0) (size 1.5 1.5) (drill 0.8) (layers "*.Cu" "*.Mask") (net "AGND"))
+  )
+  (footprint "Capacitor_SMD:C_0603" (at 150 120) (layer "F.Cu") (uuid "c_adau_100n")
+    (pad "1" smd rect (at -0.75 0) (size 0.8 0.8) (layers "F.Cu" "F.Paste" "F.Mask") (net "+3V3"))
+    (pad "2" smd rect (at 0.75 0) (size 0.8 0.8) (layers "F.Cu" "F.Paste" "F.Mask") (net "AGND"))
+  )
+  (footprint "Capacitor_THT:CP_Radial_D6.3mm_P2.50mm" (at 155 120) (layer "F.Cu") (uuid "c_adau_10u")
+    (pad "1" tht rect (at -1.25 0) (size 1.5 1.5) (drill 0.8) (layers "*.Cu" "*.Mask") (net "+3V3"))
+    (pad "2" tht oval (at 1.25 0) (size 1.5 1.5) (drill 0.8) (layers "*.Cu" "*.Mask") (net "AGND"))
+  )
+  ;; Mounting Holes
+  (footprint "MountingHole:MountingHole_3.2mm_M3" (at 45 45) (layer "F.Cu") (uuid "mh1") (pad "" tht circle (at 0 0) (size 6 6) (drill 3.2) (layers "*.Cu" "*.Mask") (net "AGND")))
+  (footprint "MountingHole:MountingHole_3.2mm_M3" (at 415 45) (layer "F.Cu") (uuid "mh2") (pad "" tht circle (at 0 0) (size 6 6) (drill 3.2) (layers "*.Cu" "*.Mask") (net "PGND")))
+  (footprint "MountingHole:MountingHole_3.2mm_M3" (at 45 165) (layer "F.Cu") (uuid "mh3") (pad "" tht circle (at 0 0) (size 6 6) (drill 3.2) (layers "*.Cu" "*.Mask") (net "AGND")))
+  (footprint "MountingHole:MountingHole_3.2mm_M3" (at 415 165) (layer "F.Cu") (uuid "mh4") (pad "" tht circle (at 0 0) (size 6 6) (drill 3.2) (layers "*.Cu" "*.Mask") (net "PGND")))
   ;; --- Full Thermal Via Array (Example for Satellite Amp) ---
   (via (at 250 60) (size 1.0) (drill 0.5) (net "PGND")) (via (at 251.5 60) (size 1.0) (drill 0.5) (net "PGND"))
@@
   ;; ... more vias to form a complete 4x3 grid ...
   ;; --- Ground Planes with Star Ground ---
-  (zone (net "AGND") (layer "B.Cu") (polygon ...))
-  (zone (net "PGND") (layer "B.Cu") (polygon ...))
-  ;; Star ground bridge: a single, wide trace on B.Cu connecting the two zones
-  (segment (start 180 100) (end 181 100) (width 3.0) (layer "B.Cu") (net "GND_BRIDGE"))
+  ;; AGND Zone (Input and Digital Section)
+  (zone (net "AGND") (layer "B.Cu") (polygon (pts (xy 40 40) (xy 181 40) (xy 181 170) (xy 40 170))))
+  ;; PGND Zone (Power Section)
+  (zone (net "PGND") (layer "B.Cu") (polygon (pts (xy 179 40) (xy 420 40) (xy 420 170) (xy 179 170))))
+  ;; Star ground bridge: Net-Tie component at X=180
+  (footprint "NetTie:NetTie-2_SMD_Pad2.0mm" (at 180 100) (layer "B.Cu") (uuid "nt_star_gnd")
+    (pad "1" smd rect (at -1.5 0) (size 2 2) (layers "B.Cu" "B.Mask") (net "AGND"))
+    (pad "2" smd rect (at 1.5 0) (size 2 2) (layers "B.Cu" "B.Mask") (net "PGND"))
+  )
   ;; --- Routing Guides on Dwgs.User Layer ---
   ;; PVDD Trace Guide
@@
   (gr_line (start 102 51) (end 148 68) (layer "Dwgs.User") (width 0.2) (stroke "dash"))
   (gr_text "Route Audio Signal. Width: 0.3mm. Keep away from power." (at 120 40) (layer "Dwgs.User"))
+  ;; --- Edge Cuts ---
+  (gr_poly (pts (xy 40 40) (xy 420 40) (xy 420 170) (xy 40 170)) (layer "Edge.Cuts") (width 0.1))
 )
